File: mcu.kicad_sch (KiCad schematic)
At the start: 40 parts, among them Q404 AO3400A, SW400 TL2243, U400 STM32H750VBTx, X300 Q13FC1350000400, X400 X322512MSB4SI

Commit message: Change MCU to STM32H563
Parts:
- removed BZ400: Buzzer, BUZ-BD12:BUZ-TH_BD12.0-P7.60-D0.6-FD, symbol Device:Buzzer
- removed C403, C407, C409, C415, C416: 100nF, PCM_JLCPCB:C_0402, symbol PCM_JLCPCB-Capacitors:0402,100nF,(2)
- removed C406, C408: 10uF, PCM_JLCPCB:C_0402, symbol PCM_JLCPCB-Capacitors:0402,10uF
- removed C411, C412: 22pF, PCM_JLCPCB:C_0402, symbol PCM_JLCPCB-Capacitors:0402,22pF
- removed C413, C414: 2.2uF, PCM_JLCPCB:C_0402, symbol PCM_JLCPCB-Capacitors:0402,2.2uF
- removed FB400: ~, PCM_JLCPCB:FB_0603, symbol PCM_JLCPCB-Inductors:Ferrite,0603
- removed R400, R401, R407: 1kΩ, PCM_JLCPCB:R_0402, symbol PCM_JLCPCB-Resistors:0402,1kΩ
- removed R403, R405: 10kΩ, PCM_JLCPCB:R_0402, symbol PCM_JLCPCB-Resistors:0402,10kΩ
- removed R404, R406: 100Ω, PCM_JLCPCB:R_0402, symbol PCM_JLCPCB-Resistors:0402,100Ω
- removed R408: 470Ω, PCM_JLCPCB:R_0402, symbol PCM_JLCPCB-Resistors:0402,470Ω
- removed R409, R433: 120Ω, PCM_JLCPCB:R_0402, symbol PCM_JLCPCB-Resistors:0402,120Ω
- removed U400: STM32H750VBTx, Package_QFP:LQFP-100_14x14mm_P0.5mm, symbol MCU_ST_STM32H7:STM32H750VBTx
- removed X400: X322512MSB4SI, PCM_JLCPCB:CRYSTAL-SMD_4P-L3.2-W2.5-BL, symbol PCM_JLCPCB-Crystals:Crystal, 12MHz, 20pF
- added BZ401: Buzzer, BUZ-BD12:BUZ-TH_BD12.0-P7.60-D0.6-FD, symbol Device:Buzzer
- added C403, C423, C425: 10uF, PCM_JLCPCB:C_0402, symbol PCM_JLCPCB-Capacitors:0402,10uF
- added C406, C417, C419, C420, C421, C422, C424, C426, C432: 100nF, PCM_JLCPCB:C_0402, symbol PCM_JLCPCB-Capacitors:0402,100nF,(2)
- added C427, C429: 2.2uF, PCM_JLCPCB:C_0402, symbol PCM_JLCPCB-Capacitors:0402,2.2uF
- added FB401: ~, PCM_JLCPCB:FB_0603, symbol PCM_JLCPCB-Inductors:Ferrite,0603
- added R434, R435, R439: 10kΩ, PCM_JLCPCB:R_0402, symbol PCM_JLCPCB-Resistors:0402,10kΩ
- added R436, R438: 100Ω, PCM_JLCPCB:R_0402, symbol PCM_JLCPCB-Resistors:0402,100Ω
- added R437: 1kΩ, PCM_JLCPCB:R_0402, symbol PCM_JLCPCB-Resistors:0402,1kΩ
- added R440, R441, R442, R443: 220Ω, PCM_JLCPCB:R_0402, symbol PCM_JLCPCB-Resistors:0402,220Ω
- added R445: 120Ω, PCM_JLCPCB:R_0402, symbol PCM_JLCPCB-Resistors:0402,120Ω
- added U405: STM32H562VGTx, Package_QFP:LQFP-100_14x14mm_P0.5mm, symbol MCU_ST_STM32H5:STM32H562VGTx
- added Y400: ASE-xxxMHz, Oscillator:Oscillator_SMD_Abracon_ASE-4Pin_3.2x2.5mm, symbol Oscillator:ASE-xxxMHz
- BTN400: renamed from SW400; LCSC C273515 -> (none)
- C313, C314: Stock 619102 -> 408081
- C400: Price 0.009USD -> 0.008USD; Stock 3940889 -> 1226257
- C401, C402, C404, C405: Stock 8389599 -> 5436546
- C410: Stock 4366811 -> 1633861
- R402: Attrition Qty 10 -> 0; Minimum Qty 20 -> 5; Stock 24372091 -> 13746052
- X300: Price 0.182USD -> 0.188USD; Stock 736610 -> 407326
Connections:
- net +3V3: now also C403.1, C406.1, C420.1, C421.1, C422.1, C425.1, C426.1, C432.1, FB401.2, R434.1, R435.1, R440.1, U405.100 (VDD), U405.11 (VDD), U405.21 (VREF+), U405.28 (VDD), U405.50 (VDD), U405.6 (VBAT), U405.73 (VDDUSB), U405.75 (VDD), Y400.1 (EN), Y400.4 (Vdd)
- net +5V: now also R445.1
- net ADS1115/RDY: now also U405.16 (PC1)
- net BOOT0: now also R437.2, R439.1, U405.94 (BOOT0); no longer R402.1
- net BOOT_EN: now also R437.1, U405.93 (PB7)
- net Buzzer: now also R402.1, U405.17 (PC2)
- net CAN1.RX: now also U405.81 (PD0)
- net CAN1.TX: now also U405.82 (PD1)
- net CAN2.RX: now also U405.51 (PB12)
- net CAN2.TX: now also U405.52 (PB13)
- net GND: now also C403.2, C406.2, C417.2, C419.2, C420.2, C421.2, C422.2, C423.2, C424.2, C425.2, C426.2, C427.2, C429.2, C432.2, R439.2, U405.10 (VSS), U405.19 (VSSA), U405.20 (VREF-), U405.27 (VSS), U405.49 (VSS), U405.74 (VSS), U405.99 (VSS), Y400.2 (GND)
- net I2C1.SCL: now also U405.95 (PB8)
- net I2C1.SDA: now also U405.96 (PB9)
- net MASTER_ON: now also U405.15 (PC0)
- net NRST: now also C419.1, R435.2, R436.1
- net ON-OFF0: now also U405.78 (PC10)
- net ON-OFF1: now also U405.79 (PC11)
- net ON-OFF2: now also U405.80 (PC12)
- net OSC32_IN: now also U405.8 (PC14)
- net OSC32_OUT: now also U405.9 (PC15)
- net OSC_IN: now also U405.12 (PH0), Y400.3 (OUT)
- net PowerButton: now also U405.63 (PC6)
- net QSPI1.CS: now also U405.47 (PB10)
- net QSPI1.IO0: now also U405.58 (PD11)
- net QSPI1.IO1: now also U405.59 (PD12)
- net QSPI1.IO2: now also U405.1 (PE2)
- net QSPI1.IO3: now also U405.60 (PD13)
- net QSPI1.SCLK: now also U405.37 (PB2)
- net STATUS_LED: now also R441.1, U405.4 (PE5)
- net SWD.SWCLK: now also U405.76 (PA14(JTCK)
- net SWD.SWDIO: now also U405.72 (PA13(JTMS)
- net SWD.~{RST}: now also R436.2, U405.14 (NRST)
- net USB_MCU.D+: now also U405.71 (PA12)
- net USB_MCU.D-: now also U405.70 (PA11)
- net USER_LED_1: now also R442.1, U405.2 (PE3)
- net USER_LED_2: now also R443.1, U405.3 (PE4)
- net USR_BTN: now also C417.1, R434.2, R438.1
- net USR_BUTTON: now also R438.2, U405.5 (PE6)
- net VCAP_1: now also C427.1, U405.48 (VCAP)
- net VCAP_2: now also C429.1, U405.98 (VCAP)
- net at Q404.3 (D): now also BZ401.2 (-)
- net at LED301.3: now also R440.2
- net at LED300.1: now also R442.2
- net at LED301.1: now also R441.2
- net at LED300.3: now also R443.2
- new net: BZ401.1 (+), R445.2
- new net STLINK.RX: U405.23 (PA0)
- new net STLINK.TX: U405.24 (PA1)
- new net VDDA: C423.1, C424.1, FB401.1, U405.22 (VDDA)
- no-connect marks 51 -> 47
Other:
- note added: "AVDD"
- note added: "Buzzer"
- note added: "CAN"
- note added: "Design choice due: es0565, sec 2.2.3"
- note added: "NOTE: PLACE CAPACTITOR AT PWR PIN"
- note added: "UART FLIP HERE"
- note removed: "C = (CL - 4pF) * 2"
- moved on the sheet: BTN400A, BTN400B, C313, C314, C410
